File: sacredHeart.brd (EAGLE design)
At the start: 57.2 x 47.4 mm, 33 parts, among them IC1 MCP73831/OT, J1 105017-0001, SW1 SPST_TACT-KMR2, U1 ATMEGA32U4-AUR, U2 SPX3819-3.3, Y1 8MHz

Commit message: Add files via upload
Connections:
- net +3V3: now also JP2.1; no longer JP2.2
- net 1: now also JP3.8; no longer JP3.2
- net 10: now also JP1.1; no longer JP1.4
- net 2: now also JP2.7; no longer JP3.1
- net 8: now also JP1.3; no longer JP1.6
- net 9: now also JP1.2; no longer JP1.5
- net A0: now also JP3.6; no longer JP3.8
- net A1: now also JP3.5; no longer JP3.7
- net A2: now also JP3.4; no longer JP3.6
- net A3: now also JP3.3; no longer JP3.5
- net A4: now also JP3.2; no longer JP3.4
- net A5: now also JP3.1; no longer JP3.3
- net AREF: now also JP3.7; no longer JP2.3
- net EN: now also JP1.5; no longer JP1.2
- net GND: now also JP2.8; no longer JP2.4
- net INT4: now also JP2.2; no longer JP1.10
- net INT5: now also JP1.11; no longer JP1.9
- net INT6: now also JP1.12; no longer JP1.8
- net INT7: now also JP2.3; no longer JP1.7
- net MISO: now also JP1.7; no longer JP2.8
- net MOSI: now also JP1.8; no longer JP2.7
- net RST: now also JP2.4; no longer JP2.1
- net SCL: now also JP2.5; no longer JP1.12
- net SCLK: now also JP1.9; no longer JP2.6
- net SDA: now also JP2.6; no longer JP1.11
- net SS: now also JP1.10; no longer JP2.5
- net VBAT: now also JP1.4; no longer JP1.1
- net VBUS: now also JP1.6; no longer JP1.3
Routing:
- net GND: track 116.8 -> 170.7 mm, vias 7 -> 5
- net SDA: track 48.4 -> 9.16 mm, vias 2 -> 0
- net SCL: track 50.4 -> 11.5 mm, vias 2 -> 0
- net RST: track 85.9 -> 58.9 mm, vias 3 -> 2
- net INT4: track 54.8 -> 31.5 mm, vias 4 -> 2
- net INT7: track 37.9 -> 15.5 mm, vias 3 -> 0
- net SS: track 19.9 -> 42.3 mm, vias 0 -> 2
- net 1: track 26.4 -> 7.26 mm, vias 2 -> 1
- net MOSI: track 22.0 -> 39.0 mm, vias 0 -> 2
- net AREF: track 74.0 -> 57.8 mm, vias 2 -> 3
- net EN: track 48.4 -> 63.9 mm, vias 4 -> 5
- net VBAT: track 81.9 -> 68.3 mm, vias 7 -> 6
- net MISO: track 24.3 -> 37.5 mm, vias 0 -> 2
- net 2: track 21.1 -> 8.09 mm
- net SCLK: track 27.5 -> 40.5 mm, vias 0 -> 2
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Other:
- board text added: "+3V3"
- board text added: "1"
- board text added: "10"
- board text added: "2"
- board text added: "8"
- board text added: "9"
- board text added: "A0"
- board text added: "A1"
- board text added: "A2"
- board text added: "A3"
- board text added: "A4"
- board text added: "A5"
- board text added: "ARF"
- board text added: "ATmega32u4 3.7V/4.2V LiPoly"
- board text added: "EN"
- board text added: "GND"
- board text added: "INT4"
- board text added: "INT5"
- board text added: "INT6"
- board text added: "INT7"
- board text added: "MISO"
- board text added: "MOSI"
- board text added: "RST"
- board text added: "SCL"
- board text added: "SCLK"
- board text added: "SDA"
- board text added: "SS"
- board text added: "SacredHeart"
- board text added: "VBAT"
- board text added: "VBUS"
