File: sacredHeart.sch (EAGLE design)
At the start: 33 parts, among them IC1 MCP73831/OT, J1 105017-0001, SW1 SPST_TACT-KMR2, U1 ATMEGA32U4-AUR, U2 SPX3819-3.3, Y1 8MHz

Commit message: Add files via upload
Connections:
- net +3V3: now also JP2.1; no longer JP2.2
- net 1: now also JP3.8; no longer JP3.2
- net 10: now also JP1.1; no longer JP1.4
- net 2: now also JP2.7; no longer JP3.1
- net 8: now also JP1.3; no longer JP1.6
- net 9: now also JP1.2; no longer JP1.5
- net A0: now also JP3.6; no longer JP3.8
- net A1: now also JP3.5; no longer JP3.7
- net A2: now also JP3.4; no longer JP3.6
- net A3: now also JP3.3; no longer JP3.5
- net A4: now also JP3.2; no longer JP3.4
- net A5: now also JP3.1; no longer JP3.3
- net AREF: now also JP3.7; no longer JP2.3
- net EN: now also JP1.5; no longer JP1.2
- net GND: now also JP2.8; no longer JP2.4
- net INT4: now also JP2.2; no longer JP1.10
- net INT5: now also JP1.11; no longer JP1.9
- net INT6: now also JP1.12; no longer JP1.8
- net INT7: now also JP2.3; no longer JP1.7
- net MISO: now also JP1.7; no longer JP2.8
- net MOSI: now also JP1.8; no longer JP2.7
- net RST: now also JP2.4; no longer JP2.1
- net SCL: now also JP2.5; no longer JP1.12
- net SCLK: now also JP1.9; no longer JP2.6
- net SDA: now also JP2.6; no longer JP1.11
- net SS: now also JP1.10; no longer JP2.5
- net VBAT: now also JP1.4; no longer JP1.1
- net VBUS: now also JP1.6; no longer JP1.3
Other:
- moved on the sheet: JP3
